File: kicad_files/rpi-shutdown-v0.kicad_pcb (KiCad board)
At the start: 2 copper layers, 86.4 x 41.9 mm, 19 parts, among them IC1 ATTINY85-S, K1 Relay_SPDT, K2 Relay_SPDT, P1 5V in, P2 Live, P3 Neutral, P4 Serial, Q1 Q_NMOS_GDS, Q2 Q_NMOS_GDS, SW1 Switch_DPST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

Commit message: Added gerbers
Routing:
- added copper zone on B.Cu, net GND
- added copper zone on F.Cu, net GND
Other:
- board text added: "git.io/vwhom"
Changed lines of the file:
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@@
     (area 40.5278 35.484999 127.351201 77.545001)
     (thickness 1.6)
-    (drawings 19)
+    (drawings 20)
     (tracks 130)
     (zones 0)
@@
     (user_trace_width 3.2512)
     (trace_clearance 0.2032)
-    (zone_clearance 3.5)
+    (zone_clearance 3)
     (zone_45_only yes)
     (trace_min 0.2032)
@@
     (visible_elements FFFFFF7F)
     (pcbplotparams
-      (layerselection 0x00030_80000001)
-      (usegerberextensions false)
+      (layerselection 0x010f0_80000001)
+      (usegerberextensions true)
       (excludeedgelayer true)
       (linewidth 0.100000)
@@
       (outputformat 1)
       (mirror false)
-      (drillshape 1)
+      (drillshape 0)
       (scaleselection 1)
-      (outputdirectory ""))
+      (outputdirectory gerbers/))
   )
   (net 0 "")
@@
     (fp_circle (center 0 0) (end 0 -2.286) (layer F.SilkS) (width 0.15))
     (pad 1 thru_hole circle (at 0 0) (size 3.2 3.2) (drill 3.2) (layers *.Cu *.Mask F.SilkS))
+  )
+  (gr_text git.io/vwhom (at 63.5 43.18) (layer F.SilkS)
+    (effects (font (size 1.5 1.5) (thickness 0.3)))
   )
   (gr_text "Version 0.1" (at 63.5 40.64) (layer F.SilkS)
@@
     (min_thickness 0.254)
     (keepout (tracks not_allowed) (vias not_allowed) (copperpour not_allowed))
-    (fill (arc_segments 16) (thermal_gap 0.508) (thermal_bridge_width 0.508))
+    (fill yes (arc_segments 16) (thermal_gap 0.508) (thermal_bridge_width 0.508))
     (polygon
       (pts
@@
     (min_thickness 0.254)
     (keepout (tracks not_allowed) (vias not_allowed) (copperpour not_allowed))
-    (fill (arc_segments 16) (thermal_gap 0.508) (thermal_bridge_width 0.508))
+    (fill yes (arc_segments 16) (thermal_gap 0.508) (thermal_bridge_width 0.508))
     (polygon
       (pts
@@
     (min_thickness 0.254)
     (keepout (tracks not_allowed) (vias not_allowed) (copperpour not_allowed))
-    (fill (arc_segments 16) (thermal_gap 0.508) (thermal_bridge_width 0.508))
+    (fill yes (arc_segments 16) (thermal_gap 0.508) (thermal_bridge_width 0.508))
     (polygon
       (pts
@@
   )
   (zone (net 13) (net_name "Net-(K1-Pad3)") (layer B.Cu) (hatch full 0.508)
-    (connect_pads yes (clearance 3.5))
+    (connect_pads yes (clearance 3))
     (min_thickness 0.254)
     (fill yes (arc_segments 16) (thermal_gap 0.508) (thermal_bridge_width 0.508))
@@
   )
   (zone (net 13) (net_name "Net-(K1-Pad3)") (layer F.Cu) (hatch full 0.508)
-    (connect_pads yes (clearance 3.5))
+    (connect_pads yes (clearance 3))
     (min_thickness 0.254)
     (fill yes (arc_segments 16) (thermal_gap 0.508) (thermal_bridge_width 0.508))
@@
     (min_thickness 0.254)
     (keepout (tracks not_allowed) (vias not_allowed) (copperpour not_allowed))
-    (fill (arc_segments 16) (thermal_gap 0.508) (thermal_bridge_width 0.508))
+    (fill yes (arc_segments 16) (thermal_gap 0.508) (thermal_bridge_width 0.508))
     (polygon
       (pts
@@
   )
   (zone (net 17) (net_name "Net-(K2-Pad3)") (layer B.Cu) (hatch full 0.508)
-    (connect_pads yes (clearance 3.5))
+    (connect_pads yes (clearance 3))
     (min_thickness 0.254)
     (fill yes (arc_segments 16) (thermal_gap 0.508) (thermal_bridge_width 0.508))
@@
       )
     )
+  )
+  (zone (net 2) (net_name GND) (layer F.Cu) (hatch full 0.508)
+    (connect_pads (clearance 0.254))
+    (min_thickness 0.254)
+    (fill yes (arc_segments 16) (thermal_gap 0.508) (thermal_bridge_width 0.508))
+    (polygon
+      (pts
+        (xy 86.36 77.47) (xy 87.63 77.47) (xy 87.63 35.56) (xy 40.64 35.56) (xy 40.64 77.47)
+      )
+    )
+  )
+  (zone (net 2) (net_name GND) (layer B.Cu) (hatch full 0.508)
+    (connect_pads (clearance 0.254))
+    (min_thickness 0.254)
+    (fill yes (arc_segments 16) (thermal_gap 0.508) (thermal_bridge_width 0.508))
+    (polygon
+      (pts
+        (xy 86.36 77.528247) (xy 87.63 77.528247) (xy 87.63 35.618247) (xy 40.64 35.618247) (xy 40.64 77.528247)
+      )
+    )

Commit message: Added gerbers and cleaned up silkscreen
Parts:
- C1, C3, C4: value C_Small -> 100nF
- C2: value CP_Small -> 10uF
- P4: value Serial -> serial
- Q1, Q2: value Q_NMOS_GDS -> FDN339AN
Changed lines of the file:
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@@
     (links 32)
     (no_connects 0)
-    (area 40.5278 35.484999 127.351201 77.545001)
+    (area 40.564999 35.484999 127.075001 77.545001)
     (thickness 1.6)
     (drawings 20)
@@
     (descr "module 1 pin (ou trou mecanique de percage)")
     (tags DEV)
-    (fp_text reference REF** (at 0 -3.048) (layer F.SilkS)
-      (effects (font (size 1 1) (thickness 0.15)))
-    )
-    (fp_text value 1pin (at 0 2.794) (layer F.Fab)
+    (fp_text reference REF** (at 0 -3.048) (layer F.SilkS) hide
+      (effects (font (size 1 1) (thickness 0.15)))
+    )
+    (fp_text value 1pin (at 0 2.794) (layer F.Fab) hide
       (effects (font (size 1 1) (thickness 0.15)))
     )
@@
     (tags "capacitor 1206")
     (attr smd)
-    (fp_text reference C1 (at 0 -2.3 180) (layer F.SilkS)
-      (effects (font (size 1 1) (thickness 0.15)))
-    )
-    (fp_text value C_Small (at 0 2.3 180) (layer F.Fab)
+    (fp_text reference C1 (at -4.445 0 180) (layer F.SilkS)
+      (effects (font (size 1 1) (thickness 0.15)))
+    )
+    (fp_text value 100nF (at 0 2.3 180) (layer F.Fab)
       (effects (font (size 1 1) (thickness 0.15)))
     )
@@
     (at 59.69 51.435 270)
     (attr smd)
-    (fp_text reference C2 (at 0 0 270) (layer F.SilkS)
-      (effects (font (size 1 1) (thickness 0.15)))
-    )
-    (fp_text value CP_Small (at 0 0 270) (layer F.Fab)
+    (fp_text reference C2 (at 3.937 0 360) (layer F.SilkS)
+      (effects (font (size 1 1) (thickness 0.15)))
+    )
+    (fp_text value 10uF (at 0 0 270) (layer F.Fab)
       (effects (font (size 1 1) (thickness 0.15)))
     )
@@
     (tags "capacitor 1206")
     (attr smd)
-    (fp_text reference C3 (at 0 -2.3 270) (layer F.SilkS)
-      (effects (font (size 1 1) (thickness 0.15)))
-    )
-    (fp_text value C_Small (at 0 2.3 270) (layer F.Fab)
+    (fp_text reference C3 (at 4.445 0 360) (layer F.SilkS)
+      (effects (font (size 1 1) (thickness 0.15)))
+    )
+    (fp_text value 100nF (at -5.969 0.508 360) (layer F.Fab)
       (effects (font (size 1 1) (thickness 0.15)))
     )
@@
     (tags "capacitor 1206")
     (attr smd)
-    (fp_text reference C4 (at 0 -2.3) (layer F.SilkS)
-      (effects (font (size 1 1) (thickness 0.15)))
-    )
-    (fp_text value C_Small (at 0 2.3) (layer F.Fab)
+    (fp_text reference C4 (at -4.191 0.254 90) (layer F.SilkS)
+      (effects (font (size 1 1) (thickness 0.15)))
+    )
+    (fp_text value 100nF (at 0 2.3) (layer F.Fab)
       (effects (font (size 1 1) (thickness 0.15)))
     )
@@
     (tags "SOIC 1.27")
     (attr smd)
-    (fp_text reference IC1 (at 0 -3.68) (layer F.SilkS)
-      (effects (font (size 1 1) (thickness 0.15)))
-    )
-    (fp_text value ATTINY85-S (at 0 3.68) (layer F.Fab)
+    (fp_text reference IC1 (at 0 3.81) (layer F.SilkS)
+      (effects (font (size 1 1) (thickness 0.15)))
+    )
+    (fp_text value ATTINY85-S (at -0.635 5.08) (layer F.Fab)
       (effects (font (size 1 1) (thickness 0.15)))
     )
@@
       (effects (font (size 1 1) (thickness 0.15)))
     )
-    (fp_text value Serial (at 2.779 7.747) (layer F.SilkS)
+    (fp_text value serial (at 2.779 7.747) (layer F.SilkS)
       (effects (font (size 1 1) (thickness 0.15)))
     )
@@
     (tags SOT-23)
     (attr smd)
-    (fp_text reference Q1 (at 0 -3.81) (layer F.SilkS)
-      (effects (font (size 1 1) (thickness 0.15)))
-    )
-    (fp_text value Q_NMOS_GDS (at -0.127 3.81) (layer F.Fab)
+    (fp_text reference Q1 (at 2.667 -1.905) (layer F.SilkS)
+      (effects (font (size 1 1) (thickness 0.15)))
+    )
+    (fp_text value FDN339AN (at -0.127 3.81) (layer F.Fab)
       (effects (font (size 1 1) (thickness 0.15)))
     )
@@
       (effects (font (size 1 1) (thickness 0.15)))
     )
-    (fp_text value Q_NMOS_GDS (at 0 3.81) (layer F.Fab)
+    (fp_text value FDN339AN (at 0 3.81) (layer F.Fab)
       (effects (font (size 1 1) (thickness 0.15)))
     )
@@
     (tags "resistor 0603")
     (attr smd)
-    (fp_text reference R2 (at 0 -1.9 90) (layer F.SilkS)
+    (fp_text reference R2 (at 2.636778 -0.110616 180) (layer F.SilkS)
       (effects (font (size 1 1) (thickness 0.15)))
     )
@@
     (tags "dpak TO-252")
     (attr smd)
-    (fp_text reference U1 (at 0 -10.414 90) (layer F.SilkS)
-      (effects (font (size 1 1) (thickness 0.15)))
-    )
-    (fp_text value AP1117D33 (at 0 -2.413 90) (layer F.Fab)
+    (fp_text reference U1 (at 4.191 -6.604 180) (layer F.SilkS)
+      (effects (font (size 1 1) (thickness 0.15)))
+    )
+    (fp_text value AP1117D33 (at 5.461 -6.35 180) (layer F.Fab)
       (effects (font (size 1 1) (thickness 0.15)))
     )
@@
     (descr "module 1 pin (ou trou mecanique de percage)")
     (tags DEV)
-    (fp_text reference REF** (at 0 -3.048) (layer F.SilkS)
-      (effects (font (size 1 1) (thickness 0.15)))
-    )
-    (fp_text value 1pin (at 0 2.794) (layer F.Fab)
+    (fp_text reference REF** (at 0 -3.048) (layer F.SilkS) hide
+      (effects (font (size 1 1) (thickness 0.15)))
+    )
+    (fp_text value 1pin (at 0 2.794) (layer F.Fab) hide
       (effects (font (size 1 1) (thickness 0.15)))
     )
@@
   (segment (start 45.72 55.2958) (end 45.72 51.435) (width 0.8128) (layer F.Cu) (net 1))
   (segment (start 47.5742 57.15) (end 45.72 55.2958) (width 0.8128) (layer F.Cu) (net 1))
+  (segment (start 76.374 67.945) (end 76.374 57.832) (width 0.4064) (layer F.Cu) (net 2))
+  (segment (start 76.374 57.832) (end 75.946 57.404) (width 0.4064) (layer F.Cu) (net 2))
+  (via (at 75.946 57.404) (size 0.7366) (drill 0.3302) (layers F.Cu B.Cu) (net 2))
+  (segment (start 75.946 57.404) (end 71.628 53.086) (width 0.4064) (layer B.Cu) (net 2))
   (segment (start 78.994 49.022) (end 79.997222 48.018778) (width 0.4064) (layer F.Cu) (net 2))
   (segment (start 79.997222 48.018778) (end 80.882616 48.018778) (width 0.4064) (layer F.Cu) (net 2))
@@
   (via (at 78.74 54.102) (size 0.7366) (drill 0.3302) (layers F.Cu B.Cu) (net 2))
   (segment (start 63.754 53.086) (end 61.341 53.086) (width 0.4064) (layer F.Cu) (net 2))
-  (segment (start 75.946 57.404) (end 71.628 53.086) (width 0.4064) (layer B.Cu) (net 2))
   (segment (start 71.628 53.086) (end 63.754 53.086) (width 0.4064) (layer B.Cu) (net 2))
   (via (at 63.754 53.086) (size 0.7366) (drill 0.3302) (layers F.Cu B.Cu) (net 2))
-  (segment (start 76.374 67.945) (end 76.374 57.832) (width 0.4064) (layer F.Cu) (net 2))
-  (segment (start 76.374 57.832) (end 75.946 57.404) (width 0.4064) (layer F.Cu) (net 2))
-  (via (at 75.946 57.404) (size 0.7366) (drill 0.3302) (layers F.Cu B.Cu) (net 2))
   (segment (start 80.899 55.669) (end 84.30786 55.669) (width 0.4064) (layer F.Cu) (net 2))
   (segment (start 84.30786 55.669) (end 84.709 55.26786) (width 0.4064) (layer F.Cu) (net 2))
